Commit message: renew submodule

File: hunter/hunter2_base/urdf/hunter2_base_gazebo.xacro (robot description, xacro)
@@ -3,6 +3,5 @@
      Commit Version: 1.6.0-1-g15f4949  Build Version: 1.6.7594.29634
      For more information, please see http://wiki.ros.org/sw_urdf_exporter -->
-<robot
-  name="hunter2_base">
+<robot xmlns:xacro="http://ros.org/wiki/xacro" name="hunter_arm">
   <link
     name="base_link">
@@ -12,5 +11,5 @@
         rpy="0 0 0" />
       <mass
-        value="1.02945169536679" />
+        value="0.02945169536679" />
       <inertia
         ixx="0.0332370959804736"
@@ -29,9 +28,9 @@
           filename="package://hunter2_base/meshes/base_link.STL" />
       </geometry>
-      <material
+      <!--material
         name="">
         <color
           rgba="0.792156862745098 0.819607843137255 0.933333333333333 1" />
-      </material>
+      </material!-->
     </visual>
     <collision>
@@ -108,12 +107,12 @@
         rpy="0 0 0" />
       <mass
-        value="0.7007" />
-      <inertia
-        ixx="0.063724"
-        ixy="-3.8745E-08"
-        ixz="2.2753E-07"
-        iyy="0.063724"
-        iyz="-4.88E-08"
-        izz="0.11072" />
+        value="7.007" />
+      <inertia
+        ixx="0.63724"
+        ixy="-3.8745E-07"
+        ixz="2.2753E-06"
+        iyy="0.63724"
+        iyz="-4.88E-07"
+        izz="1.1072" />
     </inertial>
     <visual>
@@ -125,9 +124,9 @@
           filename="package://hunter2_base/meshes/front_left_wheel_link.STL" />
       </geometry>
-      <material
-        name="">
-        <color
-          rgba="0.79216 0.81961 0.93333 1" />
-      </material>
+      <!--material
+        name="">
+        <color
+          rgba="0.79216 0.81961 0.93333 1" />
+      </material!-->
     </visual>
     <collision>
@@ -217,12 +216,12 @@
         rpy="0 0 0" />
       <mass
-        value="0.5613" />
-      <inertia
-        ixx="0.063626"
-        ixy="-6.4092E-08"
-        ixz="-2.0164E-08"
-        iyy="0.063626"
-        iyz="6.4721E-08"
-        izz="0.11054" />
+        value="5.613" />
+      <inertia
+        ixx="0.63626"
+        ixy="-6.4092E-07"
+        ixz="-2.0164E-07"
+        iyy="0.63626"
+        iyz="6.4721E-07"
+        izz="1.1054" />
     </inertial>
     <visual>
@@ -270,12 +269,12 @@
         rpy="0 0 0" />
       <mass
-        value="0.6692" />
-      <inertia
-        ixx="0.063699"
-        ixy="-2.542E-07"
-        ixz="2.638E-08"
-        iyy="0.063699"
-        iyz="-5.9934E-08"
-        izz="0.11067" />
+        value="6.692" />
+      <inertia
+        ixx="0.63699"
+        ixy="-2.542E-06"
+        ixz="2.638E-07"
+        iyy="0.63699"
+        iyz="-5.9934E-07"
+        izz="1.1067" />
     </inertial>
     <visual>
@@ -328,12 +327,12 @@
         rpy="0 0 0" />
       <mass
-        value="0.7133" />
-      <inertia
-        ixx="0.06373"
-        ixy="2.5408E-07"
-        ixz="2.6379E-08"
-        iyy="0.06373"
-        iyz="5.9941E-08"
-        izz="0.11073" />
+        value="7.133" />
+      <inertia
+        ixx="0.6373"
+        ixy="2.5408E-06"
+        ixz="2.6379E-07"
+        iyy="0.6373"
+        iyz="5.9941E-07"
+        izz="1.1073" />
     </inertial>
     <visual>
@@ -437,5 +436,5 @@
   <link
     name="rear_wheel_link">
-<inertial>
+    <inertial>
       <origin
         xyz="-0.02 0.0031269 -0.12735"
@@ -485,4 +484,55 @@
     <axis
       xyz="0 0 1" />
+  </joint>
+  <link
+    name="box_link">
+    <inertial>
+      <origin
+        xyz="0 0 0"
+        rpy="0 0 0" />
+      <mass
+        value="1" />
+      <inertia
+        ixx="0"
+        ixy="0"
+        ixz="0"
+        iyy="0"
+        iyz="0"
+        izz="0" />
+    </inertial>
+    <visual>
+      <origin
+        xyz="0 0 0"
+        rpy="0 0 0" />
+      <geometry>
+        <mesh
+          filename="package://hunter2_base/meshes/box.STL" />
+      </geometry>
+      <material
+        name="">
+        <color
+          rgba="0.79216 0.81961 0.93333 1" />
+      </material>
+    </visual>
+    <collision>
+      <origin
+        xyz="0 0 0"
+        rpy="0 0 0" />
+      <geometry>
+        <mesh
+          filename="package://hunter2_base/meshes/box.STL" />
+      </geometry>
+    </collision>
+  </link>
+  <joint
+    name="box_joint"
+    type="fixed">
+    <origin
+      xyz="0.1 0 0.11"
+      rpy="0 0 0" />
+    <parent
+      link="base_link" />
+    <child
+      link="box_link" />
   </joint>
   <gazebo reference="front_left_wheel_link">
@@ -499,8 +549,37 @@
       </gazebo>
   <gazebo>
-    <plugin name="gazebo_ros_control" filename="libgazebo_ros_control.so">
+    <plugin name="hunter_gazebo_ros_control" filename="libgazebo_ros_control.so">
       <robotSimType>steer_bot_hardware_gazebo/SteerBotHardwareGazebo</robotSimType>
-      <legacyModeNS>false</legacyModeNS>
+      <legacyModeNS>true</legacyModeNS>
     </plugin>
   </gazebo>
+  <!-- load lite6 robot -->
+  <!--joint
+    name="hunter_arm_joint"
+    type="fixed">
+    <origin
+      xyz='-0 0.35 0' rpy='0 0 3.14159265' />
+    <parent
+      link="base_link" />
+    <child
+      link="world" />
+  </joint-->
+  <xacro:include filename="$(find xarm_description)/urdf/lite6_robot_macro.xacro" />
+  <xacro:lite6_robot prefix="" namespace="ufactory" limited="false"
+    attach_to="base_link"
+    xyz='-0.35 0 0' rpy='0 0 3.14159265'
+    effort_control="false" velocity_control="false"
+    rs_d435i="true"
+    load_gazebo_plugin="true"
+    add_other_geometry="false"
+    geometry_type="box" geometry_mass="0.1"
+    geometry_height="0.1" geometry_radius="0.1"
+    geometry_length="0.1" geometry_width="0.1"
+    geometry_mesh_filename=""
+    geometry_mesh_origin_xyz="0 0 0" geometry_mesh_origin_rpy="0 0 0"
+    geometry_mesh_tcp_xyz="0 0 0" geometry_mesh_tcp_rpy="0 0 0" />
+  <xacro:include filename="$(find xarm_gripper)/urdf/xarm_gripper_model.xacro" />
+  <xacro:load_gripper attach_to="link_eef" effort_control="false" velocity_control="false" robot_dof="6" />
+  <xacro:include filename="$(find xarm_description)/urdf/camera_d435.gazebo.xacro" />
+  <xacro:realsense_d435 sensor_name="d435" rate="10"/>
 </robot>
